Commit message: change size

File: my_robot/urdf/my_robot.xacro (robot description, xacro)
@@ -2,14 +2,14 @@
 <robot name="my_robot" xmlns:xacro="http://www.ros.org/wiki/xacro">
   <gazebo reference="left_wheel">
+    <material>Gazebo/Red</material>
+  </gazebo>
+  <gazebo reference="right_wheel">
+    <material>Gazebo/Red</material>
+  </gazebo>
+  <gazebo reference="camera">
     <material>Gazebo/Green</material>
   </gazebo>
-  <gazebo reference="right_wheel">
-    <material>Gazebo/Green</material>
-  </gazebo>
-  <gazebo reference="camera">
-    <material>Gazebo/Red</material>
-  </gazebo>
   <gazebo reference="chassis">
-    <material>Gazebo/Blue</material>
+    <material>Gazebo/Orange</material>
   </gazebo>
   <xacro:include filename="$(find my_robot)/urdf/my_robot.gazebo" />
@@ -33,5 +33,5 @@
       <origin xyz="0.0 0 0" rpy=" 0 1.5707 1.5707"/>
       <geometry>
-        <cylinder radius="0.1" length="0.05"/>
+        <cylinder radius="0.12" length="0.05"/>
       </geometry>
     </collision>
@@ -39,10 +39,10 @@
       <origin xyz="0.0 0 0" rpy=" 0 1.5707 1.5707"/>
       <geometry>
-        <cylinder radius="0.1" length="0.05"/>
+        <cylinder radius="0.12" length="0.05"/>
       </geometry>
     </visual>
   </link>
   <joint type="continuous" name="right_wheel_hinge">
-    <origin xyz="0 -0.15 0" rpy="0 0 0"/>
+    <origin xyz="0 -0.175 0" rpy="0 0 0"/>
     <child link="right_wheel"/>
     <parent link="chassis"/>
@@ -64,5 +64,5 @@
       <origin xyz="0.0 0 0" rpy=" 0 1.5707 1.5707"/>
       <geometry>
-        <cylinder radius="0.1" length="0.05"/>
+        <cylinder radius="0.12" length="0.05"/>
       </geometry>
     </collision>
@@ -70,10 +70,10 @@
       <origin xyz="0.0 0 0" rpy=" 0 1.5707 1.5707"/>
       <geometry>
-        <cylinder radius="0.1" length="0.05"/>
+        <cylinder radius="0.12" length="0.05"/>
       </geometry>
     </visual>
   </link>
   <joint type="continuous" name="left_wheel_hinge">
-    <origin xyz="0 0.15 0" rpy="0 0 0"/>
+    <origin xyz="0 0.175 0" rpy="0 0 0"/>
     <child link="left_wheel"/>
     <parent link="chassis"/>
@@ -136,5 +136,5 @@
   </link>
   <joint type="fixed" name="hokuyo_joint">
-    <origin xyz="0.15 0 .1" rpy="0 0 0"/>
+    <origin xyz="0.15 0 0.075" rpy="0 0 0"/>
     <child link="hokuyo"/>
     <parent link="chassis"/>
@@ -155,5 +155,5 @@
       <origin xyz="0 0 0" rpy=" 0 0 0"/>
       <geometry>
-        <box size=".4 .2 .1"/>
+        <box size=".4 .3 .1"/>
       </geometry>
     </collision>
@@ -161,29 +161,29 @@
       <origin xyz="0 0 0" rpy=" 0 0 0"/>
       <geometry>
-        <box size=".4 .2 .1"/>
+        <box size=".4 .3 .1"/>
       </geometry>
     </visual>
     <collision name='back_caster_collision'>
-      <origin xyz="-0.15 0 -0.05" rpy=" 0 0 0"/>
+      <origin xyz="-0.12 0 -0.06" rpy=" 0 0 0"/>
       <geometry>
-        <sphere radius="0.0499"/>
+        <sphere radius="0.0599"/>
       </geometry>
     </collision>
     <visual name='back_caster_visual'>
-      <origin xyz="-0.15 0 -0.05" rpy=" 0 0 0"/>
+      <origin xyz="-0.12 0 -0.06" rpy=" 0 0 0"/>
       <geometry>
-        <sphere radius="0.05"/>
+        <sphere radius="0.06"/>
       </geometry>
     </visual>
     <collision name='front_caster_collision'>
-      <origin xyz="0.15 0 -0.05" rpy=" 0 0 0"/>
+      <origin xyz="0.12 0 -0.06" rpy=" 0 0 0"/>
       <geometry>
-        <sphere radius="0.0499"/>
+        <sphere radius="0.0599"/>
       </geometry>
     </collision>
     <visual name='front_caster_visual'>
-      <origin xyz="0.15 0 -0.05" rpy=" 0 0 0"/>
+      <origin xyz="0.12 0 -0.06" rpy=" 0 0 0"/>
       <geometry>
-        <sphere radius="0.05"/>
+        <sphere radius="0.06"/>
       </geometry>
     </visual>

Commit message: change to cylindar

File: my_robot/urdf/my_robot.xacro (robot description, xacro)
@@ -33,5 +33,5 @@
       <origin xyz="0.0 0 0" rpy=" 0 1.5707 1.5707"/>
       <geometry>
-        <cylinder radius="0.12" length="0.05"/>
+        <cylinder radius="0.05" length="0.05"/>
       </geometry>
     </collision>
@@ -39,10 +39,10 @@
       <origin xyz="0.0 0 0" rpy=" 0 1.5707 1.5707"/>
       <geometry>
-        <cylinder radius="0.12" length="0.05"/>
+        <cylinder radius="0.05" length="0.05"/>
       </geometry>
     </visual>
   </link>
   <joint type="continuous" name="right_wheel_hinge">
-    <origin xyz="0 -0.175 0" rpy="0 0 0"/>
+    <origin xyz="0 -0.25 -0.05" rpy="0 0 0"/>
     <child link="right_wheel"/>
     <parent link="chassis"/>
@@ -64,5 +64,5 @@
       <origin xyz="0.0 0 0" rpy=" 0 1.5707 1.5707"/>
       <geometry>
-        <cylinder radius="0.12" length="0.05"/>
+        <cylinder radius="0.05" length="0.05"/>
       </geometry>
     </collision>
@@ -70,10 +70,10 @@
       <origin xyz="0.0 0 0" rpy=" 0 1.5707 1.5707"/>
       <geometry>
-        <cylinder radius="0.12" length="0.05"/>
+        <cylinder radius="0.05" length="0.05"/>
       </geometry>
     </visual>
   </link>
   <joint type="continuous" name="left_wheel_hinge">
-    <origin xyz="0 0.175 0" rpy="0 0 0"/>
+    <origin xyz="0 0.25 -0.05" rpy="0 0 0"/>
     <child link="left_wheel"/>
     <parent link="chassis"/>
@@ -107,5 +107,5 @@
   </link>
   <joint type="fixed" name="camera_joint">
-    <origin xyz="0.2 0 0" rpy="0 0 0"/>
+    <origin xyz="0.28 0 0" rpy="0 0 0"/>
     <child link="camera"/>
     <parent link="chassis"/>
@@ -136,5 +136,5 @@
   </link>
   <joint type="fixed" name="hokuyo_joint">
-    <origin xyz="0.15 0 0.075" rpy="0 0 0"/>
+    <origin xyz="0.25 0 0.075" rpy="0 0 0"/>
     <child link="hokuyo"/>
     <parent link="chassis"/>
@@ -155,5 +155,5 @@
       <origin xyz="0 0 0" rpy=" 0 0 0"/>
       <geometry>
-        <box size=".4 .3 .1"/>
+        <cylinder radius="0.3" length="0.1"/>
       </geometry>
     </collision>
@@ -161,29 +161,29 @@
       <origin xyz="0 0 0" rpy=" 0 0 0"/>
       <geometry>
-        <box size=".4 .3 .1"/>
+        <cylinder radius="0.3" length="0.1"/>
       </geometry>
     </visual>
     <collision name='back_caster_collision'>
-      <origin xyz="-0.12 0 -0.06" rpy=" 0 0 0"/>
+      <origin xyz="-0.12 0 -0.05" rpy=" 0 0 0"/>
       <geometry>
-        <sphere radius="0.0599"/>
+        <sphere radius="0.0499"/>
       </geometry>
     </collision>
     <visual name='back_caster_visual'>
-      <origin xyz="-0.12 0 -0.06" rpy=" 0 0 0"/>
+      <origin xyz="-0.12 0 -0.05" rpy=" 0 0 0"/>
       <geometry>
-        <sphere radius="0.06"/>
+        <sphere radius="0.05"/>
       </geometry>
     </visual>
     <collision name='front_caster_collision'>
-      <origin xyz="0.12 0 -0.06" rpy=" 0 0 0"/>
+      <origin xyz="0.12 0 -0.05" rpy=" 0 0 0"/>
       <geometry>
-        <sphere radius="0.0599"/>
+        <sphere radius="0.0499"/>
       </geometry>
     </collision>
     <visual name='front_caster_visual'>
-      <origin xyz="0.12 0 -0.06" rpy=" 0 0 0"/>
+      <origin xyz="0.12 0 -0.05" rpy=" 0 0 0"/>
       <geometry>
-        <sphere radius="0.06"/>
+        <sphere radius="0.05"/>
       </geometry>
     </visual>

Commit message: Map My Wrold

File: my_robot/urdf/my_robot.xacro (robot description, xacro)
@@ -112,4 +112,11 @@
     <axis xyz="0 1 0" rpy="0 0 0"/>
   </joint>
+  <joint type="fixed" name="camera_optical_joint">
+    <origin xyz="0 0 0" rpy="-1.5707 0 -1.5707"/>
+    <parent link="camera"/>
+    <child link="camera_link_optical"/>
+  </joint>
+  <link name="camera_link_optical">
+  </link>
   <link name="hokuyo">
     <inertial>
